Commit message: rename primitive_objects to model.urdf

File: pybullet_object_models/primitive_objects/block/model.urdf (robot description, URDF)
Before this commit: robot block.urdf, 1 links, 0 joints
Links:
- link block: geometry collision mesh filename=block_rounded.obj scale=1.0 1.0 1.0; visual mesh filename=block_rounded.obj scale=1.0 1.0 1.0

File: pybullet_object_models/primitive_objects/cone/model.urdf (robot description, URDF)
Before this commit: robot cone.urdf, 1 links, 0 joints
Links:
- link cone: geometry collision mesh filename=cone_rounded.obj scale=1.0 1.0 1.0; visual mesh filename=cone_rounded.obj scale=1.0 1.0 1.0

File: pybullet_object_models/primitive_objects/cube/model.urdf (robot description, URDF)
Before this commit: robot cube.urdf, 1 links, 0 joints
Links:
- link cube: geometry collision mesh filename=cube_rounded.obj scale=1.0 1.0 1.0; visual mesh filename=cube_rounded.obj scale=1.0 1.0 1.0

File: pybullet_object_models/primitive_objects/cylinder/model.urdf (robot description, URDF)
Before this commit: robot cylinder.urdf, 1 links, 0 joints
Links:
- link cylinder: geometry collision mesh filename=cylinder_rounded.obj scale=1.0 1.0 1.0; visual mesh filename=cylinder_rounded.obj scale=1.0 1.0 1.0

File: pybullet_object_models/primitive_objects/dodecahedron/model.urdf (robot description, URDF)
Before this commit: robot dodecahedron.urdf, 1 links, 0 joints
Links:
- link dodecahedron: geometry collision mesh filename=dodecahedron_rounded.obj scale=1.0 1.0 1.0; visual mesh filename=dodecahedron_rounded.obj scale=1.0 1.0 1.0

File: pybullet_object_models/primitive_objects/ellipsoid/model.urdf (robot description, URDF)
Before this commit: robot ellipsoid.urdf, 1 links, 0 joints
Links:
- link ellipsoid: geometry collision mesh filename=ellipsoid_rounded.obj scale=1.0 1.0 1.0; visual mesh filename=ellipsoid_rounded.obj scale=1.0 1.0 1.0

File: pybullet_object_models/primitive_objects/hexagonal_prism/model.urdf (robot description, URDF)
Before this commit: robot hexagonal_prism.urdf, 1 links, 0 joints
Links:
- link hexagonal_prism: geometry collision mesh filename=hexagonal_prism_rounded.obj scale=1.0 1.0 1.0; visual mesh filename=hexagonal_prism_rounded.obj scale=1.0 1.0 1.0

File: pybullet_object_models/primitive_objects/hexagonal_pyramid/model.urdf (robot description, URDF)
Before this commit: robot hexagonal_pyramid.urdf, 1 links, 0 joints
Links:
- link hexagonal_pyramid: geometry collision mesh filename=hexagonal_pyramid_rounded.obj scale=1.0 1.0 1.0; visual mesh filename=hexagonal_pyramid_rounded.obj scale=1.0 1.0 1.0

File: pybullet_object_models/primitive_objects/icosahedron/model.urdf (robot description, URDF)
Before this commit: robot icosahedron.urdf, 1 links, 0 joints
Links:
- link icosahedron: geometry collision mesh filename=icosahedron_rounded.obj scale=1.0 1.0 1.0; visual mesh filename=icosahedron_rounded.obj scale=1.0 1.0 1.0

File: pybullet_object_models/primitive_objects/octagonal_prism/model.urdf (robot description, URDF)
Before this commit: robot octagonal_prism.urdf, 1 links, 0 joints
Links:
- link octagonal_prism: geometry collision mesh filename=octagonal_prism_rounded.obj scale=1.0 1.0 1.0; visual mesh filename=octagonal_prism_rounded.obj scale=1.0 1.0 1.0

File: pybullet_object_models/primitive_objects/octahedron/model.urdf (robot description, URDF)
Before this commit: robot octahedron.urdf, 1 links, 0 joints
Links:
- link octahedron: geometry collision mesh filename=octahedron_rounded.obj scale=1.0 1.0 1.0; visual mesh filename=octahedron_rounded.obj scale=1.0 1.0 1.0

File: pybullet_object_models/primitive_objects/ovaloid/model.urdf (robot description, URDF)
Before this commit: robot ovaloid.urdf, 1 links, 0 joints
Links:
- link ovaloid: geometry collision mesh filename=ovaloid_rounded.obj scale=1.0 1.0 1.0; visual mesh filename=ovaloid_rounded.obj scale=1.0 1.0 1.0

File: pybullet_object_models/primitive_objects/sphere/model.urdf (robot description, URDF)
Before this commit: robot sphere.urdf, 1 links, 0 joints
Links:
- link sphere: geometry collision mesh filename=sphere_rounded.obj scale=1.0 1.0 1.0; visual mesh filename=sphere_rounded.obj scale=1.0 1.0 1.0

File: pybullet_object_models/primitive_objects/tetrahedron/model.urdf (robot description, URDF)
Before this commit: robot tetrahedron.urdf, 1 links, 0 joints
Links:
- link empty: geometry collision mesh filename=tetrahedron_rounded.obj scale=1.0 1.0 1.0; visual mesh filename=tetrahedron_rounded.obj scale=1.0 1.0 1.0

File: pybullet_object_models/primitive_objects/torus/model.urdf (robot description, URDF)
Before this commit: robot torus.urdf, 1 links, 0 joints
Links:
- link torus: geometry collision mesh filename=torus_col.obj scale=1.0 1.0 1.0; visual mesh filename=torus_rounded.obj scale=1.0 1.0 1.0

File: pybullet_object_models/primitive_objects/triangular_prism/model.urdf (robot description, URDF)
Before this commit: robot triangular_prism.urdf, 1 links, 0 joints
Links:
- link triangular_prism: geometry collision mesh filename=triangular_prism_rounded.obj scale=1.0 1.0 1.0; visual mesh filename=triangular_prism_rounded.obj scale=1.0 1.0 1.0
